Commit message: yes1

File: final-project-tiltcontrol/description/urdf/tiltcontrol.urdf.xacro (robot description, xacro)
@@ -201,5 +201,5 @@
   <link name="pendulum">
     <inertial>
-      <origin xyz="0 0 0.15" rpy="0 0 0" />
+      <origin xyz="0 0.15 0" rpy="0 0 0" />
       <mass value="${pendulum_mass}" />
       <inertia ixx="${pendulum_ixx}" ixy="0" ixz="0" iyy="${pendulum_ixx}" iyz="0"
@@ -223,6 +223,6 @@
   </link>
   <!-- Joint from chasis to pendulum -->
-  <joint name="pendulum_joint" type="revolute">
-    <origin xyz="-0.253944 -0.05 0.17757" rpy="-1.5708 -0.214745 -3.14159"/>
+  <joint name="pendulum_joint" type="continuous">
+    <origin xyz="-0.253944 -0.05 0.17757" rpy="-1.5708 0 -3.14159"/>
     <parent link="chasis"/>
     <child link="pendulum"/>
@@ -285,4 +285,5 @@
       name="gz::sim::systems::JointStatePublisher">
       <joint_name>rail_to_cart</joint_name>
+      <joint_name>pendulum_joint</joint_name>
       <topic>/cart_joint_states</topic>
       <update_rate>100</update_rate>
